File: D22.kicad_pcb (KiCad board)
At the start: 6 copper layers, 15 x 11 mm, 48 parts, among them IC1 AVR64DD28-I_STX, IC2 NCP730BM, IC3 DRV8231ADSGR, J1 Conn_02x08_Counter_Clockwise, J2 Conn_01x01, J3 Conn_01x01, J4 Conn_01x01, Q1 BC847BDW1, Q2 BC857BDW1, Q3 PMZB200UNEYL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

Commit message: add: fuses
Parts:
- R13: value 3.3k -> 1k
Changed lines of the file:
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@@
   (title_block
     (title "RTB D22 Plux16 Decoder")
-    (date 2024-11-18)
+    (date 2025-04-20)
     (rev 0)
     (company "Frank Schumacher")
@@
     (add_net M2)
     (add_net "Net-(D3-Pad2)")
+    (add_net "Net-(IC1-Pad22)")
     (add_net "Net-(IC2-Pad2)")
+    (add_net "Net-(IC2-Pad4)")
+    (add_net "Net-(IC2-Pad5)")
     (add_net "Net-(IC3-Pad1)")
     (add_net "Net-(J1-Pad15)")
     (add_net "Net-(J1-Pad16)")
+    (add_net "Net-(J1-Pad7)")
     (add_net "Net-(Q1-Pad1)")
     (add_net "Net-(Q1-Pad5)")
@@
     (tags "Integrated Circuit")
     (attr smd)
-    (fp_text reference IC3 (at 0 0) (layer B.Fab)
+    (fp_text reference IC3 (at 0 0) (layer B.SilkS)
       (effects (font (size 1.27 1.27) (thickness 0.254)) (justify mirror))
     )
-    (fp_text value DRV8231ADSGR (at 3.77 0.44) (layer B.Fab)
+    (fp_text value DRV8231ADSGR (at 0 0) (layer B.Fab) hide
+      (effects (font (size 1.27 1.27) (thickness 0.254)) (justify mirror))
+    )
+    (fp_text user %R (at 0 0) (layer B.Fab)
       (effects (font (size 1.27 1.27) (thickness 0.254)) (justify mirror))
     )
@@
     (fp_line (start -1 0.5) (end -0.5 1) (layer B.Fab) (width 0.1))
     (fp_circle (center -1.4 1.4) (end -1.4 1.275) (layer B.SilkS) (width 0.25))
-    (fp_text user %R (at 0 0) (layer B.Fab)
-      (effects (font (size 1.27 1.27) (thickness 0.254)) (justify mirror))
-    )
     (pad 9 smd rect (at 0 0) (size 1 1.7) (layers B.Cu B.Paste B.Mask)
       (net 1 GND))
@@
       (effects (font (size 1.27 1.27) (thickness 0.254)) (justify mirror))
     )
-    (fp_text value BAS3007ARPPE6327HTSA1 (at 2.43 1.285) (layer B.Fab)
+    (fp_text value BAS3007ARPPE6327HTSA1 (at 0 0.225) (layer B.Fab)
       (effects (font (size 1.27 1.27) (thickness 0.254)) (justify mirror))
     )
-    (fp_line (start -1.45 1.025) (end 1.45 1.025) (layer B.Fab) (width 0.2))
-    (fp_line (start 1.45 1.025) (end 1.45 -0.275) (layer B.Fab) (width 0.2))
-    (fp_line (start 1.45 -0.275) (end -1.45 -0.275) (layer B.Fab) (width 0.2))
-    (fp_line (start -1.45 -0.275) (end -1.45 1.025) (layer B.Fab) (width 0.2))
-    (fp_line (start -2.45 2.825) (end 2.45 2.825) (layer B.CrtYd) (width 0.1))
-    (fp_line (start 2.45 2.825) (end 2.45 -2.375) (layer B.CrtYd) (width 0.1))
-    (fp_line (start 2.45 -2.375) (end -2.45 -2.375) (layer B.CrtYd) (width 0.1))
-    (fp_line (start -2.45 -2.375) (end -2.45 2.825) (layer B.CrtYd) (width 0.1))
-    (fp_line (start -1.45 0.775) (end -1.45 -0.025) (layer B.SilkS) (width 0.1))
-    (fp_line (start 1.45 0.775) (end 1.45 -0.025) (layer B.SilkS) (width 0.1))
-    (fp_line (start 1.45 -0.025) (end 1.45 -0.025) (layer B.SilkS) (width 0.1))
-    (fp_line (start -0.4 1.025) (end 0.4 1.025) (layer B.SilkS) (width 0.1))
-    (fp_line (start 0 -0.275) (end 0.4 -0.275) (layer B.SilkS) (width 0.1))
-    (fp_line (start -0.9 -1.325) (end -0.9 -1.325) (layer B.SilkS) (width 0.1))
-    (fp_line (start -0.8 -1.325) (end -0.8 -1.325) (layer B.SilkS) (width 0.1))
     (fp_arc (start -0.85 -1.325) (end -0.8 -1.325) (angle -180) (layer B.SilkS) (width 0.1))
     (fp_arc (start -0.85 -1.325) (end -0.9 -1.325) (angle -180) (layer B.SilkS) (width 0.1))
@@
       (effects (font (size 1.27 1.27) (thickness 0.254)) (justify mirror))
     )
+    (fp_line (start -0.8 -1.325) (end -0.8 -1.325) (layer B.SilkS) (width 0.1))
+    (fp_line (start -0.9 -1.325) (end -0.9 -1.325) (layer B.SilkS) (width 0.1))
+    (fp_line (start 0 -0.275) (end 0.4 -0.275) (layer B.SilkS) (width 0.1))
+    (fp_line (start -0.4 1.025) (end 0.4 1.025) (layer B.SilkS) (width 0.1))
+    (fp_line (start 1.45 -0.025) (end 1.45 -0.025) (layer B.SilkS) (width 0.1))
+    (fp_line (start 1.45 0.775) (end 1.45 -0.025) (layer B.SilkS) (width 0.1))
+    (fp_line (start -1.45 0.775) (end -1.45 -0.025) (layer B.SilkS) (width 0.1))
+    (fp_line (start -2.45 -2.375) (end -2.45 2.825) (layer B.CrtYd) (width 0.1))
+    (fp_line (start 2.45 -2.375) (end -2.45 -2.375) (layer B.CrtYd) (width 0.1))
+    (fp_line (start 2.45 2.825) (end 2.45 -2.375) (layer B.CrtYd) (width 0.1))
+    (fp_line (start -2.45 2.825) (end 2.45 2.825) (layer B.CrtYd) (width 0.1))
+    (fp_line (start -1.45 -0.275) (end -1.45 1.025) (layer B.Fab) (width 0.2))
+    (fp_line (start 1.45 -0.275) (end -1.45 -0.275) (layer B.Fab) (width 0.2))
+    (fp_line (start 1.45 1.025) (end 1.45 -0.275) (layer B.Fab) (width 0.2))
+    (fp_line (start -1.45 1.025) (end 1.45 1.025) (layer B.Fab) (width 0.2))
     (pad 4 smd rect (at -1 1.375 90) (size 0.9 0.8) (layers B.Cu B.Paste B.Mask)
       (net 16 VHBR))
@@
   )
   (module Resistor_SMD:R_0603_1608Metric (layer F.Cu)
-    (at 59.18 -47.84 180)
+    (at 59.2 -47.85 180)
     (descr "Resistor SMD 0603 (1608 Metric), square (rectangular) end terminal, IPC_7351 nominal, (Body size source: IPC-SM-782 page 72, https://www.pcb-3d.com/wordpress/wp-content/uploads/ipc-sm-782a_amendment_1_and_2.pdf), generated with kicad-footprint-generator")
     (tags resistor)
@@
       (effects (font (size 1 1) (thickness 0.15)) (justify mirror))
     )
-    (fp_text value 3.3k (at 0 -1.17 180) (layer B.Fab)
-      (effects (font (size 1 1) (thickness 0.15)) (justify mirror))
-    )
+    (fp_text value 1k (at 0 -1.17 180) (layer B.Fab)
+      (effects (font (size 1 1) (thickness 0.15)) (justify mirror))
+    )

Commit message: updated Kicad version
Other:
- net class Default removed
- net class Power removed
