File: D22cpu.kicad_sch (KiCad schematic)
At the start: 14 parts, among them IC1 AVR64DD28-I_STX, J1 Conn_02x08_Counter_Clockwise, J2 Conn_01x01, J3 Conn_01x01, J4 Conn_01x01

Commit message: mod: code cleanup
Parts:
- removed J3, J4: Conn_01x01, RTB:DummyNet-Connector, symbol Connector_Generic:Conn_01x01
- C8: value 100n -> 100n/50V; LCSC Part # (none) -> C307331
- D1, D2: LCSC Part # (none) -> C6297199
- D3: LCSC Part # (none) -> C130724
- IC1: Height 1 -> (none); LCSC Part # (none) -> C5156221; Manufacturer_Name Microchip -> (none); Manufacturer_Part_Number AVR64DD28-I/STX -> (none); Mouser Part Number 494-AVR64DD28-I/STX -> (none); Mouser Price/Stock https://www.mouser.co.uk/ProductDetail/Microchip-Technology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 -> (none)
- R1, R2: LCSC Part # (none) -> C25779
- R3: LCSC Part # (none) -> C25900
Connections:
- net VHBR: no longer J1.14 (Pin_14)
- new net CAP+: J1.14 (Pin_14)
Other:
- moved on the sheet: J2

Commit message: add: 15V LDO for backup cap
Parts:
- J2: footprint RTB:DummyNet-Connector -> RTB:Solder 0.8 x 0.5
- R21, R22: LCSC Part # (none) -> C25117
Changed lines of the file:
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@@
 	(title_block
 		(title "RTB D22 Plux16 Decoder")
-		(date "2026-06-28")
+		(date "2026-07-23")
 		(rev "1")
 		(company "Frank Schumacher")
@@
 			)
 		)
-		(property "Footprint" "RTB:DummyNet-Connector"
+		(property "Footprint" "RTB:Solder 0.8 x 0.5"
 			(at 204.47 132.08 0)
 			(hide yes)
@@
 			)
 		)
-		(property "Description" ""
+		(property "Description" "-55℃~+155℃ 470Ω 50V 62.5mW Thick Film Resistor ±1% ±100ppm/℃ 0402 Chip Resistor - Surface Mount ROHS"
 			(at 187.96 101.6 0)
 			(hide yes)
@@
 			)
 		)
-		(property "LCSC Part #" ""
+		(property "LCSC Part #" "C25117"
 			(at 187.96 101.6 90)
 			(hide yes)
@@
 			)
 		)
-		(property "Description" ""
+		(property "Description" "-55℃~+155℃ 470Ω 50V 62.5mW Thick Film Resistor ±1% ±100ppm/℃ 0402 Chip Resistor - Surface Mount ROHS"
 			(at 215.9 101.6 0)
 			(hide yes)
@@
 			)
 		)
-		(property "LCSC Part #" ""
+		(property "LCSC Part #" "C25117"
 			(at 215.9 101.6 90)
 			(hide yes)
