File: D22pwr.kicad_sch (KiCad schematic)
At the start: 25 parts, among them IC2 NCP730BM, IC3 DRV8231ADSGR, Q3 PMZB200UNEYL, Q4 PMZB200UNEYL, Q5 PMZB200UNEYL, Q6 PMZB200UNEYL

Commit message: mod: code cleanup
Parts:
- removed C4: 22u/25V, Capacitor_SMD:C_0603_1608Metric, symbol Device:C_Small
- removed C7: 10u/25V, Capacitor_SMD:C_0603_1608Metric, symbol Device:C_Small
- added D4: SM5819L2-TP, RTB:SM5819L2TP, symbol Device:D_Schottky
- added IC4: NCP730BMT1500TBG, Package_SON:WSON-6-1EP_2x2mm_P0.65mm_EP1x1.6mm, symbol RTB:NCP730BMT330TBG
- added R23: 100, Resistor_SMD:R_0603_1608Metric, symbol Device:R
- added R24: 10k, Resistor_SMD:R_0402_1005Metric, symbol Device:R
- C1, C2: value 22u/25V -> 10u/25V; LCSC Part # (none) -> C96446
- C10: LCSC Part # (none) -> C307331
- C3, C5: LCSC Part # (none) -> C59461
- C6: value 1u -> 1u/50V; LCSC Part # (none) -> C52923
- D8: Manufacturer_Name Infineon -> (none); Manufacturer_Part_Number BAS3007ARPPE6327HTSA1 -> (none); Mouser Part Number 726-BAS3007A-RPPE6 -> (none); Mouser Price/Stock https://www.mouser.co.uk/ProductDetail/Infineon-Technologie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 -> (none)
- IC2: value NCP730BM -> NCP730BMT500TBG; Height 0.8 -> (none); LCSC Part # (none) -> C892822; Manufacturer_Name ON Semiconductor -> (none); Manufacturer_Part_Number NCP730BMT330TBG -> (none); Mouser Part Number 863-NCP730BMT330TBG -> (none); Mouser Price/Stock https://www.mouser.co.uk/ProductDetail/onsemi/NCP730BMT330T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 -> (none)
- IC3: Height 0.8 -> (none); LCSC Part # (none) -> C5139865; Manufacturer_Name Texas Instruments -> (none); Manufacturer_Part_Number DRV8231ADSGR -> (none); Mouser Part Number 595-DRV8231ADSGR -> (none); Mouser Price/Stock https://www.mouser.co.uk/ProductDetail/Texas-Instruments/DR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 -> (none)
- Q3, Q4, Q5, Q6: Height 0.4 -> (none); LCSC Part # (none) -> C547292; Manufacturer_Name Nexperia -> (none); Manufacturer_Part_Number PMZB200UNEYL -> (none); Mouser Part Number 771-PMZB200UNEYL -> (none); Mouser Price/Stock https://www.mouser.co.uk/ProductDetail/Nexperia/PMZB200UNEY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 -> (none)
- R11, R12: LCSC Part # (none) -> C25744
- R13: LCSC Part # (none) -> C11702
- R14: LCSC Part # (none) -> C25767
- R15, R17: LCSC Part # (none) -> C25779
- R16, R18: LCSC Part # (none) -> C25752
- R19: LCSC Part # (none) -> C4346165
- R20: LCSC Part # (none) -> C25792
Connections:
- net GND: now also IC4.3 (GND), IC4.7 (EP), R24.1
- net VHBR: now also D4.1 (K), IC4.6 (IN)
- new net: IC4.1 (OUT), R23.2
- new net CAP+: D4.2 (A), R23.1, R24.2
- new net CAP_ENA: IC4.4 (EN)
- no-connect marks 3 -> 5
Other:
- note added: "Hack: SUSI.dat also used for CAP enable"
- moved on the sheet: C1, C2, C3, C5, D8, IC2, R11, R12

Commit message: add: 15V LDO for backup cap
Parts:
- C10: value 100n -> 100n/50V
- D8: LCSC Part # (none) -> C6430958
- R19: LCSC Part # C4346165 -> C22936
- R24: LCSC Part # (none) -> C25744
Changed lines of the file:
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@@
 	(title_block
 		(title "RTB D22 Plux16 Decoder")
-		(date "2026-06-28")
+		(date "2026-07-23")
 		(rev "1")
 		(company "Frank Schumacher")
@@
 			)
 		)
-		(property "Value" "100n"
-			(at 36.83 133.35 0)
+		(property "Value" "100n/50V"
+			(at 32.512 133.604 0)
 			(show_name no)
 			(do_not_autoplace no)
@@
 			)
 		)
-		(property "Description" "-55℃~+155℃ 1Ω 200mW Thick Film Resistor ±1% ±100ppm/℃ 0402 Chip Resistor - Surface Mount ROHS"
+		(property "Description" "-55℃~+155℃ 100mW 1Ω 75V Thick Film Resistor ±1% ±400ppm/℃ 0603 Chip Resistor - Surface Mount ROHS"
 			(at 186.69 140.97 0)
 			(hide yes)
@@
 			)
 		)
-		(property "LCSC Part #" "C4346165"
+		(property "LCSC Part #" "C22936"
 			(at 186.69 140.97 90)
 			(hide yes)
@@
 			)
 		)
-		(property "LCSC Part #" ""
+		(property "LCSC Part #" "C6430958"
 			(at 53.34 50.8 0)
 			(hide yes)
@@
 			)
 		)
-		(property "Description" ""
+		(property "Description" "-55℃~+155℃ 10kΩ 50V 62.5mW Thick Film Resistor ±1% ±100ppm/℃ 0402 Chip Resistor - Surface Mount ROHS"
 			(at 254 52.07 0)
 			(hide yes)
@@
 			)
 		)
-		(property "LCSC Part #" ""
+		(property "LCSC Part #" "C25744"
 			(at 254 52.07 90)
 			(hide yes)
