File: D22rcm.kicad_sch (KiCad schematic)
At the start: 9 parts, among them Q1 BC847BDW1, Q2 BC857BDW1

Commit message: mod: code cleanup
Parts:
- Q1: LCSC Part # (none) -> C455062
- Q2: LCSC Part # (none) -> C282521
- R10, R9: LCSC Part # (none) -> C25926
- R4: LCSC Part # (none) -> C25092
- R5, R6: LCSC Part # (none) -> C25744
- R7, R8: LCSC Part # (none) -> C25767
Changed lines of the file:
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@@
 	(title_block
 		(title "RTB D22 Plux16 Decoder")
-		(date "2024-11-18")
-		(rev "0")
+		(date "2026-06-28")
+		(rev "1")
 		(company "Frank Schumacher")
 		(comment 1 "Lok Decoder Plux16")
-		(comment 2 "D22.0")
+		(comment 2 "D22.1")
 		(comment 4 "Licensed under the Apache License, Version 2")
 	)
@@
 			)
 		)
-		(property "Description" ""
+		(property "Description" "-55℃~+155℃ 220kΩ 50V 62.5mW Thick Film Resistor ±1% ±100ppm/℃ 0402 Chip Resistor - Surface Mount ROHS"
 			(at 172.72 43.18 0)
+			(hide yes)
+			(show_name no)
+			(do_not_autoplace no)
+			(effects
+				(font
+					(size 1.27 1.27)
+				)
+			)
+		)
+		(property "LCSC Part #" "C25767"
+			(at 172.72 43.18 90)
+			(hide yes)
 			(show_name no)
 			(do_not_autoplace no)
@@
 			)
 		)
-		(property "Description" ""
+		(property "Description" "-55℃~+155℃ 50V 62.5mW 9.1kΩ Thick Film Resistor ±1% ±100ppm/℃ 0402 Chip Resistor - Surface Mount ROHS"
 			(at 184.15 43.18 0)
+			(hide yes)
+			(show_name no)
+			(do_not_autoplace no)
+			(effects
+				(font
+					(size 1.27 1.27)
+				)
+			)
+		)
+		(property "LCSC Part #" "C25926"
+			(at 184.15 43.18 90)
+			(hide yes)
 			(show_name no)
 			(do_not_autoplace no)
@@
 			)
 		)
-		(property "Description" ""
+		(property "Description" "-55℃~+155℃ 220kΩ 50V 62.5mW Thick Film Resistor ±1% ±100ppm/℃ 0402 Chip Resistor - Surface Mount ROHS"
 			(at 172.72 58.42 0)
+			(hide yes)
+			(show_name no)
+			(do_not_autoplace no)
+			(effects
+				(font
+					(size 1.27 1.27)
+				)
+			)
+		)
+		(property "LCSC Part #" "C25767"
+			(at 172.72 58.42 90)
+			(hide yes)
 			(show_name no)
 			(do_not_autoplace no)
@@
 			)
 		)
-		(property "Description" ""
+		(property "Description" "-55℃~+155℃ 50V 62.5mW 9.1kΩ Thick Film Resistor ±1% ±100ppm/℃ 0402 Chip Resistor - Surface Mount ROHS"
 			(at 184.15 58.42 0)
+			(hide yes)
+			(show_name no)
+			(do_not_autoplace no)
+			(effects
+				(font
+					(size 1.27 1.27)
+				)
+			)
+		)
+		(property "LCSC Part #" "C25926"
+			(at 184.15 58.42 90)
+			(hide yes)
 			(show_name no)
 			(do_not_autoplace no)
@@
 			)
 		)
-		(property "Description" ""
+		(property "Description" "-65℃~+150℃ 100MHz 100mA 2 PNP 200@2mA,5V 300mW 400mV@10mA,5mA 45V 5V 5uA PNP SOT-666-6 Bipolar (BJT) ROHS"
 			(at 81.28 49.53 0)
+			(hide yes)
+			(show_name no)
+			(do_not_autoplace no)
+			(effects
+				(font
+					(size 1.27 1.27)
+				)
+			)
+		)
+		(property "LCSC Part #" "C282521"
+			(at 81.28 49.53 0)
+			(hide yes)
 			(show_name no)
 			(do_not_autoplace no)
@@
 			)
 		)
-		(property "Description" ""
+		(property "Description" "-65℃~+150℃ 100MHz 100mA 2 PNP 200@2mA,5V 300mW 400mV@10mA,5mA 45V 5V 5uA PNP SOT-666-6 Bipolar (BJT) ROHS"
 			(at 73.66 59.69 0)
+			(hide yes)
+			(show_name no)
+			(do_not_autoplace no)
+			(effects
+				(font
+					(size 1.27 1.27)
+				)
+			)
+		)
+		(property "LCSC Part #" "C282521"
+			(at 73.66 59.69 0)
+			(hide yes)
 			(show_name no)
 			(do_not_autoplace no)
@@
 			)
 		)
-		(property "Description" ""
+		(property "Description" "-55℃~+155℃ 10kΩ 50V 62.5mW Thick Film Resistor ±1% ±100ppm/℃ 0402 Chip Resistor - Surface Mount ROHS"
 			(at 93.98 59.69 0)
+			(hide yes)
+			(show_name no)
+			(do_not_autoplace no)
+			(effects
+				(font
+					(size 1.27 1.27)
+				)
+			)
+		)
+		(property "LCSC Part #" "C25744"
+			(at 93.98 59.69 90)
+			(hide yes)
 			(show_name no)
 			(do_not_autoplace no)
@@
 			)
 		)
-		(property "Description" ""
+		(property "Description" "-55℃~+155℃ 22Ω 50V 62.5mW Thick Film Resistor ±1% ±100ppm/℃ 0402 Chip Resistor - Surface Mount ROHS"
 			(at 71.12 43.18 0)
+			(hide yes)
+			(show_name no)
+			(do_not_autoplace no)
+			(effects
+				(font
+					(size 1.27 1.27)
+				)
+			)
+		)
+		(property "LCSC Part #" "C25092"
+			(at 71.12 43.18 90)
+			(hide yes)
 			(show_name no)
 			(do_not_autoplace no)
@@
 			)
 		)
-		(property "Description" ""
+		(property "Description" "-65℃~+150℃ 100MHz 100mA 2 NPN 200 300mV 300mW 45V 5V 5uA NPN SOT-666-6 Bipolar (BJT) ROHS"
 			(at 66.04 76.2 0)
+			(hide yes)
+			(show_name no)
+			(do_not_autoplace no)
+			(effects
+				(font
+					(size 1.27 1.27)
+				)
+			)
+		)
+		(property "LCSC Part #" "C455062"
+			(at 66.04 76.2 0)
+			(hide yes)
 			(show_name no)
 			(do_not_autoplace no)
@@
 			)
 		)
-		(property "Description" ""
+		(property "Description" "-55℃~+155℃ 10kΩ 50V 62.5mW Thick Film Resistor ±1% ±100ppm/℃ 0402 Chip Resistor - Surface Mount ROHS"
 			(at 78.74 76.2 0)
+			(hide yes)
+			(show_name no)
+			(do_not_autoplace no)
+			(effects
+				(font
+					(size 1.27 1.27)
+				)
+			)
+		)
+		(property "LCSC Part #" "C25744"
+			(at 78.74 76.2 90)
+			(hide yes)
 			(show_name no)
 			(do_not_autoplace no)
@@
 			)
 		)
-		(property "Description" ""
+		(property "Description" "-65℃~+150℃ 100MHz 100mA 2 NPN 200 300mV 300mW 45V 5V 5uA NPN SOT-666-6 Bipolar (BJT) ROHS"
 			(at 66.04 95.25 0)
-			(show_name no)
-			(do_not_autoplace no)
+			(hide yes)
+			(show_name no)
+			(do_not_autoplace no)
+			(effects
+				(font
+					(size 1.27 1.27)
+				)
+			)
+		)
+		(property "LCSC Part #" "C455062"
+			(at 66.04 95.25 0)
+			(hide yes)
+			(show_name no)
+			(do_not_autoplace no)

Commit message: add: 15V LDO for backup cap
Parts:
- R10, R9: LCSC Part # C25926 -> C163450
Changed lines of the file:
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@@
 	(title_block
 		(title "RTB D22 Plux16 Decoder")
-		(date "2026-06-28")
+		(date "2026-07-23")
 		(rev "1")
 		(company "Frank Schumacher")
@@
 			)
 		)
-		(property "LCSC Part #" "C25926"
+		(property "LCSC Part #" " C163450"
 			(at 184.15 43.18 90)
 			(hide yes)
@@
 			)
 		)
-		(property "LCSC Part #" "C25926"
+		(property "LCSC Part #" " C163450"
 			(at 184.15 58.42 90)
 			(hide yes)
